File: hardware/industrial-dual-ac-in.kicad_pcb (KiCad board)
At the start: 2 copper layers, 40 x 40 mm, 34 parts, among them P1 CON-SENSOR2, P2 BOOT, P3 Debug, P4 Input, U1 XMC1100, U109 HCPL2731

Commit message: updated mounting holes
Parts:
- Drill1, Drill2, Drill3, Drill4: footprint kicad-libraries:DRILL_NP_35 -> kicad-libraries:DRILL_NP
Changed lines of the file:
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@@
   (net 11 "Net-(P1-Pad5)")
   (net 12 "Net-(P1-Pad6)")
-  (net 13 "Net-(U1-Pad3)")
-  (net 14 "Net-(U1-Pad2)")
+  (net 13 "Net-(P2-Pad2)")
+  (net 14 "Net-(P3-Pad1)")
   (net 15 "unconnected-(P4-Pad2)")
   (net 16 "unconnected-(P4-Pad3)")
@@
     )
     (pad "1" smd circle locked (at 0 0) (size 0.7 0.7) (layers "F.Cu" "F.Paste" "F.Mask")
-      (net 14 "Net-(U1-Pad2)") (pinfunction "P1") (pintype "passive"))
+      (net 14 "Net-(P3-Pad1)") (pinfunction "P1") (pintype "passive"))
   )
   (footprint "kicad-libraries:QFN24-4x4mm-0.5mm" (layer "F.Cu")
@@
       (net 23 "S-MISO") (pinfunction "P2.0_AIO") (pintype "passive"))
     (pad "2" smd oval locked (at -2.025 -0.75 270) (size 1 0.3) (layers "F.Cu" "F.Paste" "F.Mask")
-      (net 14 "Net-(U1-Pad2)") (pinfunction "P2.1_AIO") (pintype "passive"))
+      (net 14 "Net-(P3-Pad1)") (pinfunction "P2.1_AIO") (pintype "passive"))
     (pad "3" smd oval locked (at -2.025 -0.25 270) (size 1 0.3) (layers "F.Cu" "F.Paste" "F.Mask")
-      (net 13 "Net-(U1-Pad3)") (pinfunction "P2.2_AI") (pintype "passive"))
+      (net 13 "Net-(P2-Pad2)") (pinfunction "P2.2_AI") (pintype "passive"))
     (pad "4" smd oval locked (at -2.025 0.25 270) (size 1 0.3) (layers "F.Cu" "F.Paste" "F.Mask")
       (net 33 "unconnected-(U1-Pad4)") (pinfunction "P2.6_AI") (pintype "passive+no_connect"))
@@
       (net 9 "Net-(D116-Pad2)") (pinfunction "K") (pintype "passive"))
   )
-  (footprint "kicad-libraries:DRILL_NP_35" (layer "F.Cu")
+  (footprint "kicad-libraries:DRILL_NP" (layer "F.Cu")
     (at 102.5 97.5)
     (property "Sheetfile" "industrial-dual-ac-in.kicad_sch")
@@
     (fp_circle (center 0 0) (end 1.69926 0) (layer "B.SilkS") (width 0.381) (fill none))
     (fp_circle (center 0 0) (end 1.39954 -0.09906) (layer "B.SilkS") (width 0.381) (fill none))
+    (fp_circle (center 0 0) (end 2.19964 0) (layer "B.SilkS") (width 0.381) (fill none))
     (fp_circle (center 0 0) (end 1.89992 0) (layer "B.SilkS") (width 0.381) (fill none))
-    (fp_circle (center 0 0) (end 2.19964 0) (layer "B.SilkS") (width 0.381) (fill none))
+    (fp_circle (center 0 0) (end 1.99898 -0.20066) (layer "F.SilkS") (width 0.381) (fill none))
     (fp_circle (center 0 0) (end 1.69926 0) (layer "F.SilkS") (width 0.381) (fill none))
-    (fp_circle (center 0 0) (end 1.99898 -0.20066) (layer "F.SilkS") (width 0.381) (fill none))
     (fp_circle (center 0 0) (end 1.39954 0) (layer "F.SilkS") (width 0.381) (fill none))
     (fp_circle (center 0 0) (end 2.19964 -0.20066) (layer "F.SilkS") (width 0.381) (fill none))
     (fp_circle (center 0 0) (end 3.2 0) (layer "Eco2.User") (width 0.01) (fill none))
-    (pad "" np_thru_hole circle locked (at 0 0) (size 3.5 3.5) (drill 3.5) (layers *.Cu *.Mask "F.SilkS")
+    (pad "" np_thru_hole circle locked (at 0 0) (size 2.99974 2.99974) (drill 2.99974) (layers *.Cu *.Mask "F.SilkS")
       (clearance 0.89916))
   )
-  (footprint "kicad-libraries:DRILL_NP_35" (layer "F.Cu")
+  (footprint "kicad-libraries:DRILL_NP" (layer "F.Cu")
     (at 102.5 62.5)
     (property "Sheetfile" "industrial-dual-ac-in.kicad_sch")
@@
     )
     (fp_circle (center 0 0) (end 1.39954 -0.09906) (layer "B.SilkS") (width 0.381) (fill none))
-    (fp_circle (center 0 0) (end 1.89992 0) (layer "B.SilkS") (width 0.381) (fill none))
     (fp_circle (center 0 0) (end 2.19964 0) (layer "B.SilkS") (width 0.381) (fill none))
     (fp_circle (center 0 0) (end 1.69926 0) (layer "B.SilkS") (width 0.381) (fill none))
+    (fp_circle (center 0 0) (end 1.89992 0) (layer "B.SilkS") (width 0.381) (fill none))
     (fp_circle (center 0 0) (end 1.69926 0) (layer "F.SilkS") (width 0.381) (fill none))
     (fp_circle (center 0 0) (end 2.19964 -0.20066) (layer "F.SilkS") (width 0.381) (fill none))
@@
     (fp_circle (center 0 0) (end 1.39954 0) (layer "F.SilkS") (width 0.381) (fill none))
     (fp_circle (center 0 0) (end 3.2 0) (layer "Eco2.User") (width 0.01) (fill none))
-    (pad "" np_thru_hole circle locked (at 0 0) (size 3.5 3.5) (drill 3.5) (layers *.Cu *.Mask "F.SilkS")
+    (pad "" np_thru_hole circle locked (at 0 0) (size 2.99974 2.99974) (drill 2.99974) (layers *.Cu *.Mask "F.SilkS")
       (clearance 0.89916))
   )
@@
     )
   )
-  (footprint "kicad-libraries:DRILL_NP_35" (layer "F.Cu")
+  (footprint "kicad-libraries:DRILL_NP" (layer "F.Cu")
     (at 137.5 62.5)
     (property "Sheetfile" "industrial-dual-ac-in.kicad_sch")
@@
       (effects (font (size 0.29972 0.29972) (thickness 0.0762)))
     )
+    (fp_circle (center 0 0) (end 2.19964 0) (layer "B.SilkS") (width 0.381) (fill none))
     (fp_circle (center 0 0) (end 1.89992 0) (layer "B.SilkS") (width 0.381) (fill none))
     (fp_circle (center 0 0) (end 1.69926 0) (layer "B.SilkS") (width 0.381) (fill none))
     (fp_circle (center 0 0) (end 1.39954 -0.09906) (layer "B.SilkS") (width 0.381) (fill none))
-    (fp_circle (center 0 0) (end 2.19964 0) (layer "B.SilkS") (width 0.381) (fill none))
+    (fp_circle (center 0 0) (end 1.99898 -0.20066) (layer "F.SilkS") (width 0.381) (fill none))
     (fp_circle (center 0 0) (end 1.39954 0) (layer "F.SilkS") (width 0.381) (fill none))
     (fp_circle (center 0 0) (end 2.19964 -0.20066) (layer "F.SilkS") (width 0.381) (fill none))
-    (fp_circle (center 0 0) (end 1.99898 -0.20066) (layer "F.SilkS") (width 0.381) (fill none))
     (fp_circle (center 0 0) (end 1.69926 0) (layer "F.SilkS") (width 0.381) (fill none))
     (fp_circle (center 0 0) (end 3.2 0) (layer "Eco2.User") (width 0.01) (fill none))
-    (pad "" np_thru_hole circle locked (at 0 0) (size 3.5 3.5) (drill 3.5) (layers *.Cu *.Mask "F.SilkS")
+    (pad "" np_thru_hole circle locked (at 0 0) (size 2.99974 2.99974) (drill 2.99974) (layers *.Cu *.Mask "F.SilkS")
       (clearance 0.89916))
   )
@@
       (net 2 "GND") (pinfunction "P1") (pintype "passive"))
     (pad "2" smd rect locked (at 0.55 0 270) (size 0.3 1.4) (layers "F.Cu" "F.Mask")
-      (net 13 "Net-(U1-Pad3)") (pinfunction "P2") (pintype "passive"))
+      (net 13 "Net-(P2-Pad2)") (pinfunction "P2") (pintype "passive"))
     (pad "2" smd rect locked (at 0.15 0 270) (size 0.6 0.5) (layers "F.Cu" "F.Mask")
-      (net 13 "Net-(U1-Pad3)") (pinfunction "P2") (pintype "passive"))
+      (net 13 "Net-(P2-Pad2)") (pinfunction "P2") (pintype "passive"))
   )
   (footprint "kicad-libraries:Logo_31x31" (layer "F.Cu")
@@
     )
   )
-  (footprint "kicad-libraries:DRILL_NP_35" (layer "F.Cu")
+  (footprint "kicad-libraries:DRILL_NP" (layer "F.Cu")
     (at 137.5 97.5)
     (property "Sheetfile" "industrial-dual-ac-in.kicad_sch")
@@
     )
     (fp_circle (center 0 0) (end 1.39954 -0.09906) (layer "B.SilkS") (width 0.381) (fill none))
+    (fp_circle (center 0 0) (end 2.19964 0) (layer "B.SilkS") (width 0.381) (fill none))
+    (fp_circle (center 0 0) (end 1.89992 0) (layer "B.SilkS") (width 0.381) (fill none))
     (fp_circle (center 0 0) (end 1.69926 0) (layer "B.SilkS") (width 0.381) (fill none))
-    (fp_circle (center 0 0) (end 1.89992 0) (layer "B.SilkS") (width 0.381) (fill none))
-    (fp_circle (center 0 0) (end 2.19964 0) (layer "B.SilkS") (width 0.381) (fill none))
-    (fp_circle (center 0 0) (end 1.69926 0) (layer "F.SilkS") (width 0.381) (fill none))
     (fp_circle (center 0 0) (end 2.19964 -0.20066) (layer "F.SilkS") (width 0.381) (fill none))
     (fp_circle (center 0 0) (end 1.39954 0) (layer "F.SilkS") (width 0.381) (fill none))
+    (fp_circle (center 0 0) (end 1.69926 0) (layer "F.SilkS") (width 0.381) (fill none))
     (fp_circle (center 0 0) (end 1.99898 -0.20066) (layer "F.SilkS") (width 0.381) (fill none))
     (fp_circle (center 0 0) (end 3.2 0) (layer "Eco2.User") (width 0.01) (fill none))
-    (pad "" np_thru_hole circle locked (at 0 0) (size 3.5 3.5) (drill 3.5) (layers *.Cu *.Mask "F.SilkS")
+    (pad "" np_thru_hole circle locked (at 0 0) (size 2.99974 2.99974) (drill 2.99974) (layers *.Cu *.Mask "F.SilkS")
       (clearance 0.89916))
   )
@@
   (segment (start 106.6 61.3) (end 106.9501 60.9499) (width 0.25) (layer "F.Cu") (net 4))
   (segment (start 128.911759 61) (end 129.8 61) (width 0.3) (layer "F.Cu") (net 4))
-  (segment (start 107.55 60.9499) (end 107.2501 60.9499) (width 0.15) (layer "F.Cu") (net 4))
   (segment (start 121.15 68.8) (end 121.2 68.85) (width 0.25) (layer "F.Cu") (net 4))
   (segment (start 122.1 70.2) (end 123.711759 70.2) (width 0.3) (layer "F.Cu") (net 4))
@@
   (segment (start 104.9 68.8) (end 104.9 68.6) (width 0.5) (layer "B.Cu") (net 4))
   (segment (start 116.19 72.61) (end 116.19 74.79) (width 0.5) (layer "B.Cu") (net 4))
-  (segment (start 107.6501 62.45) (end 107.55 62.5501) (width 0.25) (layer "F.Cu") (net 5))
   (segment (start 108.95 61.05) (end 108.95 61.2501) (width 0.25) (layer "F.Cu") (net 5))
-  (segment (start 107.8001 62.7) (end 107.6501 62.55) (width 0.25) (layer "F.Cu") (net 5))
   (segment (start 108.95 61.2501) (end 107.55 62.6501) (width 0.25) (layer "F.Cu") (net 5))
   (segment (start 132.25042 91.93425) (end 132.25042 89.24958) (width 1) (layer "F.Cu") (net 6))
